File: Kicad/plantid.kicad_pcb (KiCad board)
At the start: 2 copper layers, 64.5 x 66.5 mm, 26 parts, among them J1 SMT50, J2 Pump, J3 Battery, J4 Load Mod r, J5 Load Mod l, J6 IO16-19, J7 RX/TX, J8 Spacer r, J9 Spacer l, U1 WE-TVS-824015043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

Commit message: Add files via upload
Parts:
- moved Q4 15.2 mm to (125.0, 109.2)
- moved R1 15.2 mm to (128.8, 109.2)
- renumbered U4 to Q4
Connections:
- U1 pad 3: /Temperature -> unconnected-(U1-I/O2-Pad3)
- U1 pad 6: unconnected-(U1-I/O4-Pad6) -> /Temperature
Routing:
- net GND: track 93.4 -> 20.2 mm
- net Net-(D1-A): track 32.0 -> 15.1 mm, vias 2 -> 0
- net /Gate: track 21.3 -> 7.96 mm, vias 2 -> 0
- net /Charger +: track 46.6 -> 49.9 mm, vias 4 -> 1
- net +3.3V: track 47.0 -> 44.5 mm
- net /Temperature: track 46.6 -> 47.7 mm
- net /Moisture: track 38.8 -> 39.5 mm
