File: Kicad/plantid.kicad_sch (KiCad schematic)
At the start: 26 parts, among them J1 SMT50, J2 Pump, J3 Battery, J4 Load Mod r, J5 Load Mod l, J6 IO16-19, J7 RX/TX, J8 Spacer r, J9 Spacer l, U1 WE-TVS-824015043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

Commit message: Add files via upload
Parts:
- renumbered U4 to Q4
Connections:
- net Temperature: now also U1.6 (I/O4); no longer U1.3 (I/O2)
Other:
- moved on the sheet: C7
Changed lines of the file:
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@@
   (no_connect (at 87.63 104.14))
   (no_connect (at 242.57 41.91))
+  (no_connect (at 127 153.67))
   (no_connect (at 46.99 109.22))
   (no_connect (at 87.63 86.36))
-  (no_connect (at 147.32 153.67))
   (no_connect (at 87.63 119.38))
   (no_connect (at 46.99 124.46))
@@
     (stroke (width 0) (type default))
   )
-  (wire (pts (xy 157.48 161.29) (xy 157.48 154.94))
+  (wire (pts (xy 165.1 161.29) (xy 165.1 154.94))
     (stroke (width 0) (type default))
   )
@@
     (stroke (width 0) (type default))
   )
-  (wire (pts (xy 157.48 147.32) (xy 157.48 137.16))
+  (wire (pts (xy 165.1 147.32) (xy 165.1 137.16))
     (stroke (width 0) (type default))
   )
@@
     (stroke (width 0) (type default))
   )
-  (wire (pts (xy 137.16 161.29) (xy 157.48 161.29))
+  (wire (pts (xy 137.16 161.29) (xy 165.1 161.29))
     (stroke (width 0) (type default))
   )
@@
     (stroke (width 0) (type default))
   )
-  (wire (pts (xy 157.48 137.16) (xy 137.16 137.16))
+  (wire (pts (xy 165.1 137.16) (xy 137.16 137.16))
     (stroke (width 0) (type default))
   )
@@
     (effects (font (size 1.27 1.27)) (justify left bottom))
   )
-  (label "Temperature" (at 127 153.67 180) (fields_autoplaced)
-    (effects (font (size 1.27 1.27)) (justify right bottom))
+  (label "Temperature" (at 147.32 153.67 0) (fields_autoplaced)
+    (effects (font (size 1.27 1.27)) (justify left bottom))
   )
   (label "IO18" (at 50.8 173.99 0) (fields_autoplaced)
@@
     )
   )
-  (symbol (lib_id "Device:C") (at 157.48 151.13 0) (unit 1)
-    (in_bom yes) (on_board yes) (dnp no)
-    (property "Reference" "C7" (at 151.13 151.13 0)
-      (effects (font (size 1.27 1.27)) (justify left))
-    )
-    (property "Value" "100n" (at 151.13 153.67 0)
-      (effects (font (size 1.27 1.27)) (justify left))
-    )
-    (property "Footprint" "Capacitor_SMD:C_0603_1608Metric_Pad1.08x0.95mm_HandSolder" (at 158.4452 154.94 0)
-      (effects (font (size 1.27 1.27)) hide)
-    )
-    (property "Datasheet" "~" (at 157.48 151.13 0)
-      (effects (font (size 1.27 1.27)) hide)
-    )
-    (property "Digikey" "1276-1000-1-ND" (at 157.48 151.13 0)
+  (symbol (lib_id "Device:C") (at 165.1 151.13 0) (unit 1)
+    (in_bom yes) (on_board yes) (dnp no)
+    (property "Reference" "C7" (at 158.75 151.13 0)
+      (effects (font (size 1.27 1.27)) (justify left))
+    )
+    (property "Value" "100n" (at 158.75 153.67 0)
+      (effects (font (size 1.27 1.27)) (justify left))
+    )
+    (property "Footprint" "Capacitor_SMD:C_0603_1608Metric_Pad1.08x0.95mm_HandSolder" (at 166.0652 154.94 0)
+      (effects (font (size 1.27 1.27)) hide)
+    )
+    (property "Datasheet" "~" (at 165.1 151.13 0)
+      (effects (font (size 1.27 1.27)) hide)
+    )
+    (property "Digikey" "1276-1000-1-ND" (at 165.1 151.13 0)
       (effects (font (size 1.27 1.27)) hide)
     )
@@
   (symbol (lib_id "BSH108:BSH108") (at 215.9 144.78 0) (unit 1)
     (in_bom yes) (on_board yes) (dnp no) (fields_autoplaced)
-    (property "Reference" "U4" (at 227.33 143.51 0)
+    (property "Reference" "Q4" (at 227.33 143.51 0)
       (effects (font (size 1.524 1.524)) (justify left))
     )
@@
       (project "plantid"
         (path "/c4d8de9b-2494-4722-b282-cc2d6553a774"
-          (reference "U4") (unit 1)
-        )
-      )
+          (reference "Q4") (unit 1)
+        )
+      )
